File: Marconi_2955_Step_Attenuator/Marconi_2955_Step_Attenuator.kicad_pcb (KiCad board)
At the start: 4 copper layers, 125 x 20 mm, 45 parts

Commit message: update to v1.4
Parts:
- C10, C11, C12, C13, C14, C15, C16, C17, C18, C19, C20, C21, C7, C8, C9: value 330pf -> 100nF
- R1, R2, R3, R4, R5: footprint Resistor_SMD:R_0603_1608Metric -> Resistor_SMD:R_0805_2012Metric
- renumbered OUT to J1, IN to J2, PM3 to J3
Connections:
- REF** pad 1: (no net) -> GND (x4)
Routing:
- net GND: vias 25 -> 117
Other:
- board text added: "V1.4"
- board text removed: "V1.3"
