File: Marconi_2955_Step_Attenuator/Marconi_2955_Step_Attenuator.kicad_sch (KiCad schematic)
At the start: 40 parts, among them J1 Conn_SMA, J2 Conn_SMA, J3 PM3

Commit message: update to v1.4
Parts:
- C10, C11, C12, C13, C14, C15, C16, C17, C18, C19, C20, C21, C7, C8, C9: value 330pf -> 100nF
- R1, R2, R3, R4, R5: footprint Resistor_SMD:R_0603_1608Metric -> Resistor_SMD:R_0805_2012Metric
Other:
- note added: "3x100nF"
- note removed: "3x330pF"
Changed lines of the file:
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@@
 		)
 	)
-	(text "3x330pF"
+	(text "3x100nF"
 		(exclude_from_sim no)
 		(at 69.342 74.168 0)
@@
 		)
 	)
-	(text "3x330pF"
+	(text "3x100nF"
 		(exclude_from_sim no)
 		(at 164.084 74.168 0)
@@
 		)
 	)
-	(text "3x330pF"
+	(text "3x100nF"
 		(exclude_from_sim no)
 		(at 100.838 74.168 0)
@@
 		)
 	)
-	(text "3x330pF"
+	(text "3x100nF"
 		(exclude_from_sim no)
 		(at 131.826 74.422 0)
@@
 		)
 	)
-	(text "3x330pF"
+	(text "3x100nF"
 		(exclude_from_sim no)
 		(at 195.072 74.422 0)
@@
 			)
 		)
-		(property "Value" "330pf"
+		(property "Value" "100nF"
 			(at 198.1263 76.7277 90)
 			(effects
@@
 			)
 		)
-		(property "Value" "330pf"
+		(property "Value" "100nF"
 			(at 198.1263 79.2677 90)
 			(effects
@@
 			)
 		)
-		(property "Value" "330pf"
+		(property "Value" "100nF"
 			(at 71.1263 74.1877 90)
 			(effects
@@
 			)
 		)
-		(property "Footprint" "Resistor_SMD:R_0603_1608Metric"
+		(property "Footprint" "Resistor_SMD:R_0805_2012Metric"
 			(at 148.59 69.85 0)
 			(effects
@@
 			)
 		)
-		(property "Footprint" "Resistor_SMD:R_0603_1608Metric"
+		(property "Footprint" "Resistor_SMD:R_0805_2012Metric"
 			(at 116.84 69.85 0)
 			(effects
@@
 			)
 		)
-		(property "Value" "330pf"
+		(property "Value" "100nF"
 			(at 102.8763 74.1877 90)
 			(effects
@@
 			)
 		)
-		(property "Value" "330pf"
+		(property "Value" "100nF"
 			(at 198.1263 74.1877 90)
 			(effects
@@
 			)
 		)
-		(property "Value" "330pf"
+		(property "Value" "100nF"
 			(at 102.362 73.914 90)
 			(effects
@@
 			)
 		)
-		(property "Footprint" "Resistor_SMD:R_0603_1608Metric"
+		(property "Footprint" "Resistor_SMD:R_0805_2012Metric"
 			(at 85.09 69.85 0)
 			(effects
@@
 			)
 		)
-		(property "Value" "330pf"
+		(property "Value" "100nF"
 			(at 134.6263 76.7277 90)
 			(effects
@@
 			)
 		)
-		(property "Footprint" "Resistor_SMD:R_0603_1608Metric"
+		(property "Footprint" "Resistor_SMD:R_0805_2012Metric"
 			(at 50.8 69.85 0)
 			(effects
@@
 			)
 		)
-		(property "Value" "330pf"
+		(property "Value" "100nF"
 			(at 166.3763 74.1877 90)
 			(effects
@@
 			)
 		)
-		(property "Footprint" "Resistor_SMD:R_0603_1608Metric"
+		(property "Footprint" "Resistor_SMD:R_0805_2012Metric"
 			(at 180.34 69.85 0)
 			(effects
@@
 			)
 		)
-		(property "Value" "330pf"
+		(property "Value" "100nF"
 			(at 134.6263 79.2677 90)
 			(effects
@@
 			)
 		)
-		(property "Value" "330pf"
+		(property "Value" "100nF"
 			(at 102.8763 76.7277 90)
 			(effects
@@
 			)
 		)
-		(property "Value" "330pf"
+		(property "Value" "100nF"
 			(at 71.1263 76.7277 90)
 			(effects
@@
 			)
 		)
-		(property "Value" "330pf"
+		(property "Value" "100nF"
 			(at 166.3763 79.2677 90)
 			(effects
@@
 			)
 		)
-		(property "Value" "330pf"
+		(property "Value" "100nF"
 			(at 134.6263 74.1877 90)
 			(effects
@@
 			)
 		)
-		(property "Value" "330pf"
+		(property "Value" "100nF"
 			(at 71.1263 79.2677 90)
 			(effects
@@
 			)
 		)
-		(property "Value" "330pf"
+		(property "Value" "100nF"
 			(at 166.3763 76.7277 90)
 			(effects
